Commit message: Add Working visulaization

File: Ros2_packages/diff_robot_iti/diff_robot_description/urdf/robot_control.xacro (robot description, xacro)
@@ -1,40 +1,63 @@
 <?xml version="1.0"?>
 <robot xmlns:xacro="http://www.ros.org/wiki/xacro">
+  <!-- Need to double check-->
   <xacro:property name="wheel_separation" value="0.2116"/>
-  <xacro:property name="wheel_diameter" value="0.028"/>
+  <xacro:property name="wheel_radius" value="0.0325"/>
   <xacro:property name="max_wheel_torque" value="10"/>
-  <!-- <ros2_control name="robot_hardware" type="system">
-    <hardware>
+  <!-- Real hardware / Mock for now :) -->
+  <xacro:unless value="$(arg sim_mode)">
+    <ros2_control name="RealRobot" type="system">
+   <hardware>
       <plugin>mock_components/GenericSystem</plugin>
+      <param name="calculate_dynamics">true</param>
+          <param name="disable_commands">false</param>
     </hardware>
-    <joint name="left_wheel_joint">
-      <command_interface name="velocity"/>
-      <state_interface name="position"/>
-      <state_interface name="velocity"/>
-    </joint>
-    <joint name="right_wheel_joint">
-      <command_interface name="velocity"/>
-      <state_interface name="position"/>
-      <state_interface name="velocity"/>
-    </joint>
-  </ros2_control> -->
+      <joint name="left_wheel_joint">
+        <command_interface name="velocity">
+          <param name="min">-10</param>
+          <param name="max">10</param>
+        </command_interface>
+        <state_interface name="position"/>
+        <state_interface name="velocity"/>
+      </joint>
+      <joint name="right_wheel_joint">
+        <command_interface name="velocity">
+          <param name="min">-10</param>
+          <param name="max">10</param>
+        </command_interface>
+        <state_interface name="position"/>
+        <state_interface name="velocity"/>
+      </joint>
+    </ros2_control>
+  </xacro:unless>
+  <!-- Gazebo simulation -->
+  <xacro:if value="$(arg sim_mode)">
+    <ros2_control name="GazeboSystem" type="system">
+      <hardware>
+        <plugin>gazebo_ros2_control/GazeboSystem</plugin>
+      </hardware>
+      <joint name="left_wheel_joint">
+        <command_interface name="velocity">
+          <param name="min">-10</param>
+          <param name="max">10</param>
+        </command_interface>
+        <state_interface name="velocity"/>
+        <state_interface name="position"/>
+      </joint>
+      <joint name="right_wheel_joint">
+        <command_interface name="velocity">
+          <param name="min">-10</param>
+          <param name="max">10</param>
+        </command_interface>
+        <state_interface name="velocity"/>
+        <state_interface name="position"/>
+      </joint>
+    </ros2_control>
+  </xacro:if>
+  <!-- Gazebo plugin -->
   <gazebo>
-    <plugin name="diff_drive" filename="libgazebo_ros_diff_drive.so">
-      <ros>
-        <namespace>/</namespace>
-        <remapping>cmd_vel:=cmd_vel</remapping>
-        <remapping>odom:=odom</remapping>
-      </ros>
-      <left_joint>left_wheel_joint</left_joint>
-      <right_joint>right_wheel_joint</right_joint>
-      <wheel_separation>${wheel_separation}</wheel_separation>
-      <wheel_diameter>${wheel_diameter}</wheel_diameter>
-      <max_wheel_torque>${max_wheel_torque}</max_wheel_torque>
-      <max_wheel_acceleration>1.0</max_wheel_acceleration>
-      <odometry_frame>odom</odometry_frame>
-      <robot_base_frame>base_link</robot_base_frame>
-      <publish_odom>true</publish_odom>
-      <publish_odom_tf>true</publish_odom_tf>
-      <publish_wheel_tf>false</publish_wheel_tf>
+    <plugin name="gazebo_ros2_control" filename="libgazebo_ros2_control.so">
+      <parameters>$(find diff_robot_bringup)/config/my_controllers.yaml</parameters>
+      <parameters>$(find diff_robot_bringup)/config/gaz_ros2_ctl_use_sim.yaml</parameters>
     </plugin>
   </gazebo>

File: Ros2_packages/diff_robot_iti/diff_robot_description/urdf/sensors.xacro (robot description, xacro)
@@ -21,5 +21,5 @@
   </link>
   <joint name="imu_joint" type="fixed">
-    <parent link="base_link"/>
+    <parent link="chassis_link"/>
     <child link="imu_link"/>
     <origin xyz="0.05 0 0.08" rpy="0 0 0"/>
@@ -74,5 +74,5 @@
       <geometry>
         <mesh
-          filename="package://diff_robot_description/meshes/lidar_link.STL" />
+          filename="file://$(find diff_robot_description)/meshes/lidar_link.STL" />
       </geometry>
       <material
@@ -88,5 +88,5 @@
       <geometry>
         <mesh
-          filename="package://diff_robot_description/meshes/lidar_link.STL" />
+          filename="file://$(find diff_robot_description)/meshes/lidar_link.STL" />
       </geometry>
     </collision>
@@ -99,5 +99,5 @@
       rpy="0 0 0" />
     <parent
-      link="base_link" />
+      link="chassis_link" />
     <child
       link="lidar_link" />
@@ -105,37 +105,30 @@
       xyz="0 0 0" />
   </joint>
-  <gazebo reference="lidar_link">
-    <sensor name="lidar" type="gpu_lidar">
-      <pose>0 0 0 0 0 0</pose>
-      <visualize>true</visualize>
-      <update_rate>10</update_rate>
-      <lidar>
-        <scan>
-          <horizontal>
-            <samples>360</samples>
-            <resolution>1</resolution>
-            <min_angle>${-pi}</min_angle>
-            <max_angle>${pi}</max_angle>
-          </horizontal>
-        </scan>
-        <range>
-          <min>0.12</min>
-          <max>12.0</max>
-          <resolution>0.01</resolution>
-        </range>
-        <noise>
-          <type>gaussian</type>
-          <mean>0.0</mean>
-          <stddev>0.01</stddev>
-        </noise>
-      </lidar>
-      <plugin name="lidar_plugin" filename="libgazebo_ros_lidar.so">
-        <ros>
-          <namespace>/sensors</namespace>
-          <remapping>~/out:=scan</remapping>
-        </ros>
-        <frame_name>lidar_link</frame_name>
-      </plugin>
-    </sensor>
-  </gazebo>
+   <gazebo reference="lidar_link">
+        <sensor name="laser" type="ray">
+            <pose> 0 0 0 0 0 0 </pose>
+            <visualize>true</visualize>
+            <update_rate>10</update_rate>
+            <ray>
+                <scan>
+                    <horizontal>
+                        <samples>360</samples>
+                        <min_angle>-3.14</min_angle>
+                        <max_angle>3.14</max_angle>
+                    </horizontal>
+                </scan>
+                <range>
+                    <min>0.3</min>
+                    <max>12</max>
+                </range>
+            </ray>
+            <plugin name="laser_controller" filename="libgazebo_ros_ray_sensor.so">
+                <ros>
+                    <argument>~/out:=scan</argument>
+                </ros>
+                <output_type>sensor_msgs/LaserScan</output_type>
+                <frame_name>lidar_link</frame_name>
+            </plugin>
+        </sensor>
+    </gazebo>
 </robot>

File: Ros2_packages/diff_robot_iti/diff_robot_description/urdf/solidworks_gen.xacro (robot description, xacro)
@@ -4,6 +4,14 @@
      For more information, please see http://wiki.ros.org/sw_urdf_exporter -->
 <robot xmlns:xacro="http://www.ros.org/wiki/xacro">
-  <link
-    name="base_link">
+  <!-- Dummy base_link  -->
+  <link name="base_link"/>
+  <!-- Chassis holds all SolidWorks geometry -->
+  <joint name="base_link_joint" type="fixed">
+    <parent link="base_link"/>
+    <child link="chassis_link"/>
+    <origin xyz="0 0 0" rpy="0 0 0"/>
+  </joint>
+  <link
+    name="chassis_link">
     <inertial>
       <origin
@@ -26,19 +34,19 @@
       <geometry>
         <mesh
-          filename="package://diff_robot_description/meshes/base_link.STL" />
-      </geometry>
-      <material
-        name="">
-        <color
-          rgba="0.792156862745098 0.819607843137255 0.933333333333333 1" />
-      </material>
-    </visual>
-    <collision>
-      <origin
-        xyz="0 0 0"
-        rpy="0 0 0" />
-      <geometry>
-        <mesh
-          filename="package://diff_robot_description/meshes/base_link.STL" />
+          filename="file://$(find diff_robot_description)/meshes/base_link.STL" />
+      </geometry>
+      <material
+        name="">
+        <color
+          rgba="0.792156862745098 0.819607843137255 0.933333333333333 1" />
+      </material>
+    </visual>
+    <collision>
+      <origin
+        xyz="0 0 0"
+        rpy="0 0 0" />
+      <geometry>
+        <mesh
+          filename="file://$(find diff_robot_description)/meshes/base_link.STL" />
       </geometry>
     </collision>
@@ -66,19 +74,19 @@
       <geometry>
         <mesh
-          filename="package://diff_robot_description/meshes/left_wheel_link.STL" />
-      </geometry>
-      <material
-        name="">
-        <color
-          rgba="0.792156862745098 0.819607843137255 0.933333333333333 1" />
-      </material>
-    </visual>
-    <collision>
-      <origin
-        xyz="0 0 0"
-        rpy="0 0 0" />
-      <geometry>
-        <mesh
-          filename="package://diff_robot_description/meshes/left_wheel_link.STL" />
+          filename="file://$(find diff_robot_description)/meshes/left_wheel_link.STL" />
+      </geometry>
+      <material
+        name="">
+        <color
+          rgba="0.792156862745098 0.819607843137255 0.933333333333333 1" />
+      </material>
+    </visual>
+    <collision>
+      <origin
+        xyz="0 0 0"
+        rpy="0 0 0" />
+      <geometry>
+        <mesh
+          filename="file://$(find diff_robot_description)/meshes/left_wheel_link.STL" />
       </geometry>
     </collision>
@@ -91,12 +99,12 @@
       rpy="-1.5708 0 0" />
     <parent
-      link="base_link" />
+      link="chassis_link" />
     <child
       link="left_wheel_link" />
     <axis
-      xyz="0 0 1" />
+      xyz="0 0 -1" />
     <dynamics
       damping="0.1"
-      friction="0.1" />
+      friction="2.0" />
   </joint>
   <link
@@ -122,19 +130,19 @@
       <geometry>
         <mesh
-          filename="package://diff_robot_description/meshes/right_wheel_link.STL" />
-      </geometry>
-      <material
-        name="">
-        <color
-          rgba="0.792156862745098 0.819607843137255 0.933333333333333 1" />
-      </material>
-    </visual>
-    <collision>
-      <origin
-        xyz="0 0 0"
-        rpy="0 0 0" />
-      <geometry>
-        <mesh
-          filename="package://diff_robot_description/meshes/right_wheel_link.STL" />
+          filename="file://$(find diff_robot_description)/meshes/right_wheel_link.STL" />
+      </geometry>
+      <material
+        name="">
+        <color
+          rgba="0.792156862745098 0.819607843137255 0.933333333333333 1" />
+      </material>
+    </visual>
+    <collision>
+      <origin
+        xyz="0 0 0"
+        rpy="0 0 0" />
+      <geometry>
+        <mesh
+          filename="file://$(find diff_robot_description)/meshes/right_wheel_link.STL" />
       </geometry>
     </collision>
@@ -147,5 +155,5 @@
       rpy="-1.5708 0 0" />
     <parent
-      link="base_link" />
+      link="chassis_link" />
     <child
       link="right_wheel_link" />
@@ -153,44 +161,44 @@
       xyz="0 0 -1" />
     <dynamics
-      damping="0.1"
-      friction="0.1" />
-  </joint>
-   <link
+      damping="1.1"
+      friction="2.0" />
+  </joint>
+  <link
     name="right_caster_link">
     <inertial>
       <origin
-        xyz="0.16269 -0.0033135 0.059265"
-        rpy="0 0 0" />
-      <mass
-        value="0.033269" />
-      <inertia
-        ixx="3.951E-06"
-        ixy="-1.7081E-08"
-        ixz="8.3812E-08"
-        iyy="5.9564E-06"
-        iyz="1.1147E-08"
-        izz="3.3163E-06" />
-    </inertial>
-    <visual>
-      <origin
-        xyz="0 0 0"
-        rpy="0 0 0" />
-      <geometry>
-        <mesh
-          filename="package://diff_robot_description/meshes/right_caster_link.STL" />
-      </geometry>
-      <material
-        name="">
-        <color
-          rgba="0.79216 0.81961 0.93333 1" />
-      </material>
-    </visual>
-    <collision>
-      <origin
-        xyz="0 0 0"
-        rpy="0 0 0" />
-      <geometry>
-        <mesh
-          filename="package://diff_robot_description/meshes/right_caster_link.STL" />
+        xyz="0.00268816148973561 -0.00203536418614769 0.00191349352759729"
+        rpy="0 0 0" />
+      <mass
+        value="0.0332686534414054" />
+      <inertia
+        ixx="3.95101603832686E-06"
+        ixy="8.38120688817775E-08"
+        ixz="1.70812071112867E-08"
+        iyy="3.31627423081446E-06"
+        iyz="-1.11469659665923E-08"
+        izz="5.95635417481321E-06" />
+    </inertial>
+    <visual>
+      <origin
+        xyz="0 0 0"
+        rpy="0 0 0" />
+      <geometry>
+        <mesh
+          filename="file://$(find diff_robot_description)/meshes/right_caster_link.STL" />
+      </geometry>
+      <material
+        name="">
+        <color
+          rgba="0.792156862745098 0.819607843137255 0.933333333333333 1" />
+      </material>
+    </visual>
+    <collision>
+      <origin
+        xyz="0 0 0"
+        rpy="0 0 0" />
+      <geometry>
+        <mesh
+          filename="file://$(find diff_robot_description)/meshes/right_caster_link.STL" />
       </geometry>
     </collision>
@@ -200,8 +208,8 @@
     type="fixed">
     <origin
-      xyz="-0.0713498457201036 -0.105808252244339 -0.0264000000000171"
-      rpy="-1.5707963267949 0 0" />
-    <parent
-      link="base_link" />
+      xyz="0.08865 -0.044508 -0.025"
+      rpy="0 0 0" />
+    <parent
+      link="chassis_link" />
     <child
       link="right_caster_link" />
@@ -213,37 +221,37 @@
     <inertial>
       <origin
-        xyz="0.16269 -0.0033135 -0.062773"
-        rpy="0 0 0" />
-      <mass
-        value="0.033269" />
-      <inertia
-        ixx="3.951E-06"
-        ixy="-1.7081E-08"
-        ixz="8.3812E-08"
-        iyy="5.9564E-06"
-        iyz="1.1147E-08"
-        izz="3.3163E-06" />
-    </inertial>
-    <visual>
-      <origin
-        xyz="0 0 0"
-        rpy="0 0 0" />
-      <geometry>
-        <mesh
-          filename="package://diff_robot_description/meshes/left_caster_link.STL" />
-      </geometry>
-      <material
-        name="">
-        <color
-          rgba="0.79216 0.81961 0.93333 1" />
-      </material>
-    </visual>
-    <collision>
-      <origin
-        xyz="0 0 0"
-        rpy="0 0 0" />
-      <geometry>
-        <mesh
-          filename="package://diff_robot_description/meshes/left_caster_link.STL" />
+        xyz="0.00268816148974094 -0.00147315327391973 0.00191349352759895"
+        rpy="0 0 0" />
+      <mass
+        value="0.0332686534414053" />
+      <inertia
+        ixx="3.95101603832685E-06"
+        ixy="8.38120688817571E-08"
+        ixz="1.70812071113248E-08"
+        iyy="3.31627423081444E-06"
+        iyz="-1.11469659666131E-08"
+        izz="5.95635417481318E-06" />
+    </inertial>
+    <visual>
+      <origin
+        xyz="0 0 0"
+        rpy="0 0 0" />
+      <geometry>
+        <mesh
+          filename="file://$(find diff_robot_description)/meshes/left_caster_link.STL" />
+      </geometry>
+      <material
+        name="">
+        <color
+          rgba="0.792156862745098 0.819607843137255 0.933333333333333 1" />
+      </material>
+    </visual>
+    <collision>
+      <origin
+        xyz="0 0 0"
+        rpy="0 0 0" />
+      <geometry>
+        <mesh
+          filename="file://$(find diff_robot_description)/meshes/left_caster_link.STL" />
       </geometry>
     </collision>
@@ -253,8 +261,8 @@
     type="fixed">
     <origin
-      xyz="-0.0713498457200881 0.105791747755655 -0.0263999999999989"
-      rpy="-1.5707963267949 0 0" />
-    <parent
-      link="base_link" />
+      xyz="0.08865 0.044508 -0.025"
+      rpy="0 0 0" />
+    <parent
+      link="chassis_link" />
     <child
       link="left_caster_link" />
@@ -262,3 +270,15 @@
       xyz="0 0 0" />
   </joint>
+<gazebo reference="left_wheel_link">
+  <mu1>100000000000000.0</mu1>
+  <mu2>100000000000000.0</mu2>
+  <kp>100000000000000</kp>
+  <kd>100</kd>
+</gazebo>
+<gazebo reference="right_wheel_link">
+  <mu1>100000000000000.0</mu1>
+  <mu2>100000000000000.0</mu2>
+  <kp>100000000000000</kp>
+  <kd>100</kd>
+</gazebo>
 </robot>
