Commit message: Add initial full high level system packages

File: Ros2_packages/diff_robot_iti/diff_robot_description/urdf/robot.xacro (robot description, xacro)
@@ -1,4 +1,9 @@
 <?xml version="1.0"?>
 <robot xmlns:xacro="http://www.ros.org/wiki/xacro" name="my_robot">
+  <xacro:arg name="sim_mode" default="false"/>
+  <xacro:arg name="use_mock_hardware" default="false"/>
+  <xacro:arg name="serial_device" default="/dev/ttyUSB0"/>
+  <xacro:arg name="baud_rate" default="115200"/>
+  <xacro:arg name="enc_counts_per_rev" default="340"/>
   <xacro:include filename="solidworks_gen.xacro"/>
   <xacro:include filename="sensors.xacro"/>

File: Ros2_packages/diff_robot_iti/diff_robot_description/urdf/robot_control.xacro (robot description, xacro)
@@ -1,46 +1,7 @@
 <?xml version="1.0"?>
 <robot xmlns:xacro="http://www.ros.org/wiki/xacro">
-  <xacro:arg name="use_mock_hardware" default="false"/>
-  <!-- Need to double check-->
   <xacro:property name="wheel_separation" value="0.2116"/>
   <xacro:property name="wheel_radius" value="0.0325"/>
   <xacro:property name="max_wheel_torque" value="10"/>
-  <!-- Real hardware / Mock for now :) -->
-  <xacro:unless value="$(arg sim_mode)">
-    <ros2_control name="RealRobot" type="system">
-    <hardware>
-      <xacro:if value="$(arg use_mock_hardware)">
-        <plugin>mock_components/GenericSystem</plugin>
-        <param name="calculate_dynamics">true</param>
-        <param name="disable_commands">false</param>
-      </xacro:if>
-      <xacro:unless value="$(arg use_mock_hardware)">
-        <plugin>diffdrive_hardware/DiffDriveHardwareSystem</plugin>
-        <param name="left_wheel_name">left_wheel_joint</param>
-        <param name="right_wheel_name">right_wheel_joint</param>
-        <param name="serial_device">/dev/ttyUSB0</param>
-        <param name="baud_rate">115200</param>
-        <param name="enc_counts_per_rev">340</param>
-        <param name="imu_name">imu_sensor</param>
-      </xacro:unless>
-    </hardware>
-      <joint name="left_wheel_joint">
-        <command_interface name="velocity">
-          <param name="min">-10</param>
-          <param name="max">10</param>
-        </command_interface>
-        <state_interface name="position"/>
-        <state_interface name="velocity"/>
-      </joint>
-      <joint name="right_wheel_joint">
-        <command_interface name="velocity">
-          <param name="min">-10</param>
-          <param name="max">10</param>
-        </command_interface>
-        <state_interface name="position"/>
-        <state_interface name="velocity"/>
-      </joint>
-    </ros2_control>
-  </xacro:unless>
   <!-- Gazebo simulation -->
   <xacro:if value="$(arg sim_mode)">
@@ -65,12 +26,72 @@
         <state_interface name="position"/>
       </joint>
+      <sensor name="imu_sensor">
+        <state_interface name="linear_acceleration.x"/>
+        <state_interface name="linear_acceleration.y"/>
+        <state_interface name="linear_acceleration.z"/>
+        <state_interface name="angular_velocity.x"/>
+        <state_interface name="angular_velocity.y"/>
+        <state_interface name="angular_velocity.z"/>
+        <state_interface name="orientation.x"/>
+        <state_interface name="orientation.y"/>
+        <state_interface name="orientation.z"/>
+        <state_interface name="orientation.w"/>
+      </sensor>
     </ros2_control>
+    <gazebo>
+      <plugin name="gazebo_ros2_control" filename="libgazebo_ros2_control.so">
+        <parameters>$(find diff_robot_bringup)/config/controllers.yaml</parameters>
+        <parameters>$(find diff_robot_bringup)/config/gaz_ros2_ctl_use_sim.yaml</parameters>
+      </plugin>
+    </gazebo>
   </xacro:if>
-  <!-- Gazebo plugin -->
-  <gazebo>
-    <plugin name="gazebo_ros2_control" filename="libgazebo_ros2_control.so">
-      <parameters>$(find diff_robot_bringup)/config/my_controllers.yaml</parameters>
-      <parameters>$(find diff_robot_bringup)/config/gaz_ros2_ctl_use_sim.yaml</parameters>
-    </plugin>
-  </gazebo>
+  <!-- Real hardware or Mock -->
+  <xacro:unless value="$(arg sim_mode)">
+    <ros2_control name="RealRobot" type="system">
+      <hardware>
+        <xacro:if value="$(arg use_mock_hardware)">
+          <plugin>mock_components/GenericSystem</plugin>
+          <param name="calculate_dynamics">true</param>
+          <param name="disable_commands">false</param>
+        </xacro:if>
+        <xacro:unless value="$(arg use_mock_hardware)">
+          <plugin>diffdrive_hardware/DiffDriveHardwareSystem</plugin>
+          <param name="left_wheel_name">left_wheel_joint</param>
+          <param name="right_wheel_name">right_wheel_joint</param>
+          <param name="serial_device">$(arg serial_device)</param>
+          <param name="baud_rate">$(arg baud_rate)</param>
+          <param name="enc_counts_per_rev">$(arg enc_counts_per_rev)</param>
+          <param name="imu_name">imu_sensor</param>
+        </xacro:unless>
+      </hardware>
+      <joint name="left_wheel_joint">
+        <command_interface name="velocity">
+          <param name="min">-10</param>
+          <param name="max">10</param>
+        </command_interface>
+        <state_interface name="position"/>
+        <state_interface name="velocity"/>
+      </joint>
+      <joint name="right_wheel_joint">
+        <command_interface name="velocity">
+          <param name="min">-10</param>
+          <param name="max">10</param>
+        </command_interface>
+        <state_interface name="position"/>
+        <state_interface name="velocity"/>
+      </joint>
+      <sensor name="imu_sensor">
+        <state_interface name="linear_acceleration.x"/>
+        <state_interface name="linear_acceleration.y"/>
+        <state_interface name="linear_acceleration.z"/>
+        <state_interface name="angular_velocity.x"/>
+        <state_interface name="angular_velocity.y"/>
+        <state_interface name="angular_velocity.z"/>
+        <state_interface name="orientation.x"/>
+        <state_interface name="orientation.y"/>
+        <state_interface name="orientation.z"/>
+        <state_interface name="orientation.w"/>
+      </sensor>
+    </ros2_control>
+  </xacro:unless>
 </robot>

File: Ros2_packages/diff_robot_iti/diff_robot_description/urdf/sensors.xacro (robot description, xacro)
@@ -52,83 +52,59 @@
   </gazebo>
   <!-- ==================== LIDAR ==================== -->
-   <link
-    name="lidar_link">
+  <link name="lidar_link">
     <inertial>
-      <origin
-        xyz="-0.0014514 3.2754E-06 0.019293"
-        rpy="0 0 0" />
-      <mass
-        value="0.17546" />
-      <inertia
-        ixx="8.2171E-05"
-        ixy="1.6745E-07"
-        ixz="-3.7671E-06"
-        iyy="0.00010613"
-        iyz="8.5784E-09"
-        izz="0.00014061" />
+      <origin xyz="-0.0014514 3.2754E-06 0.019293" rpy="0 0 0"/>
+      <mass value="0.17546"/>
+      <inertia ixx="8.2171E-05" ixy="1.6745E-07" ixz="-3.7671E-06"
+               iyy="0.00010613" iyz="8.5784E-09" izz="0.00014061"/>
     </inertial>
     <visual>
-      <origin
-        xyz="0 0 0"
-        rpy="${pi/2} 0 0" />
+      <origin xyz="0 0 0" rpy="${pi/2} 0 0"/>
       <geometry>
-        <mesh
-          filename="file://$(find diff_robot_description)/meshes/lidar_link.STL" />
+        <mesh filename="file://$(find diff_robot_description)/meshes/lidar_link.STL"/>
       </geometry>
-      <material
-        name="">
-        <color
-          rgba="0.79216 0.81961 0.93333 1" />
+      <material name="">
+        <color rgba="0.79216 0.81961 0.93333 1"/>
       </material>
     </visual>
     <collision>
-      <origin
-        xyz="0 0 0"
-        rpy="0 0 0" />
+      <origin xyz="0 0 0" rpy="0 0 0"/>
       <geometry>
-        <mesh
-          filename="file://$(find diff_robot_description)/meshes/lidar_link.STL" />
+        <mesh filename="file://$(find diff_robot_description)/meshes/lidar_link.STL"/>
       </geometry>
     </collision>
   </link>
-  <joint
-    name="lidar_joint"
-    type="fixed">
-    <origin
-      xyz="0.0990647710242247 0 0.0963999999999987"
-      rpy="0 0 0" />
-    <parent
-      link="chassis_link" />
-    <child
-      link="lidar_link" />
-    <axis
-      xyz="0 0 0" />
+  <joint name="lidar_joint" type="fixed">
+    <origin xyz="0.0990647710242247 0 0.0963999999999987" rpy="0 0 0"/>
+    <parent link="chassis_link"/>
+    <child link="lidar_link"/>
+    <axis xyz="0 0 0"/>
   </joint>
-   <gazebo reference="lidar_link">
-        <sensor name="laser" type="ray">
-            <pose> 0 0 0 0 0 0 </pose>
-            <visualize>true</visualize>
-            <update_rate>10</update_rate>
-            <ray>
-                <scan>
-                    <horizontal>
-                        <samples>360</samples>
-                        <min_angle>-3.14</min_angle>
-                        <max_angle>3.14</max_angle>
-                    </horizontal>
-                </scan>
-                <range>
-                    <min>0.3</min>
-                    <max>12</max>
-                </range>
-            </ray>
-            <plugin name="laser_controller" filename="libgazebo_ros_ray_sensor.so">
-                <ros>
-                    <argument>~/out:=scan</argument>
-                </ros>
-                <output_type>sensor_msgs/LaserScan</output_type>
-                <frame_name>lidar_link</frame_name>
-            </plugin>
-        </sensor>
-    </gazebo>
+  <gazebo reference="lidar_link">
+    <sensor name="laser" type="ray">
+      <pose>0 0 0 0 0 0</pose>
+      <visualize>true</visualize>
+      <update_rate>10</update_rate>
+      <ray>
+        <scan>
+          <horizontal>
+            <samples>360</samples>
+            <min_angle>-3.14</min_angle>
+            <max_angle>3.14</max_angle>
+          </horizontal>
+        </scan>
+        <range>
+          <min>0.3</min>
+          <max>12</max>
+        </range>
+      </ray>
+      <plugin name="laser_controller" filename="libgazebo_ros_ray_sensor.so">
+        <ros>
+          <argument>~/out:=scan</argument>
+        </ros>
+        <output_type>sensor_msgs/LaserScan</output_type>
+        <frame_name>lidar_link</frame_name>
+      </plugin>
+    </sensor>
+  </gazebo>
 </robot>

File: Ros2_packages/diff_robot_iti/diff_robot_description/urdf/solidworks_gen.xacro (robot description, xacro)
@@ -4,4 +4,11 @@
      For more information, please see http://wiki.ros.org/sw_urdf_exporter -->
 <robot xmlns:xacro="http://www.ros.org/wiki/xacro">
+  <!-- needed -->
+  <link name="base_footprint"/>
+  <joint name="base_footprint_joint" type="fixed">
+    <parent link="base_footprint"/>
+    <child link="base_link"/>
+    <origin xyz="0 0 0.0589" rpy="0 0 0"/>
+  </joint>
   <!-- Dummy base_link  -->
   <link name="base_link"/>
@@ -161,5 +168,5 @@
       xyz="0 0 -1" />
     <dynamics
-      damping="1.1"
+      damping="0.1"
       friction="2.0" />
   </joint>
